File: CatSatShield/CaTSatShield.sch (KiCad schematic (older format))
At the start: 5 parts, among them J1 , J2 , J3 BME280, J4 CCS811

Commit message: Routeo
Parts:
- J4: footprint Pines:62000811121 -> Pin_Headers:Pin_Header_Straight_1x07_Pitch2.54mm
Changed lines of the file:
@@
 F 0 "J4" H 8514 2232 50  0000 L CNN
 F 1 "CCS811" H 8514 2141 50  0000 L CNN
-F 2 "Pines:62000811121" H 8435 2240 50  0001 C CNN
+F 2 "Pin_Headers:Pin_Header_Straight_1x07_Pitch2.54mm" H 8435 2240 50  0001 C CNN
 F 3 "~" H 8435 2240 50  0001 C CNN
 	1    8435 2240
