File: CatSatShield/CaTSatShield.sch (KiCad schematic (older format))
At the start: 5 parts, among them J1 , J2 , J3 BME280, J4 CCS811

Commit message: Label wakeA6 sch
Parts:
- J3: footprint Pines:61300411121 -> Connector_PinSocket_2.54mm:PinSocket_1x04_P2.54mm_Vertical
Connections:
- net labels added: WAKEA6
- net labels removed: WAK-A6, WAKE-A6
Changed lines of the file:
@@
 A5
 Text Label 1530 2515 2    50   ~ 0
-WAKE-A6
+WAKEA6
 Text Label 1530 2615 2    50   ~ 0
 0
@@
 F 0 "J3" H 10440 2187 50  0000 L CNN
 F 1 "BME280" H 10440 2096 50  0000 L CNN
-F 2 "Pines:61300411121" H 10360 2195 50  0001 C CNN
+F 2 "Connector_PinSocket_2.54mm:PinSocket_1x04_P2.54mm_Vertical" H 10360 2195 50  0001 C CNN
 F 3 "~" H 10360 2195 50  0001 C CNN
 	1    10360 2195
@@
 10-INTCCS
 Text Label 8020 2340 2    50   ~ 0
-WAK-A6
+WAKEA6
 Text Label 8015 2240 0    50   ~ 0
 SDA
@@
 NoConn ~ 4640 2460
 $Comp
-L power:+3.3V #PWR?
+L power:+3.3V #PWR0102
 U 1 1 5BB2D67F
 P 8010 1940
-F 0 "#PWR?" H 8010 1790 50  0001 C CNN
+F 0 "#PWR0102" H 8010 1790 50  0001 C CNN
 F 1 "+3.3V" H 8025 2113 50  0000 C CNN
 F 2 "" H 8010 1940 50  0001 C CNN
@@
 $EndComp
 $Comp
-L power:+3.3V #PWR?
+L power:+3.3V #PWR0103
 U 1 1 5BB2D707
 P 9950 2095
-F 0 "#PWR?" H 9950 1945 50  0001 C CNN
+F 0 "#PWR0103" H 9950 1945 50  0001 C CNN
 F 1 "+3.3V" H 9965 2268 50  0000 C CNN
 F 2 "" H 9950 2095 50  0001 C CNN
